Commit message: Muevo carpetas dentro de src

File: src/my_robot_description/urdf/mobile_base.xacro (robot description, xacro)
@@ -2,7 +2,7 @@
 <robot xmlns:xacro="http://www.ros.org/wiki/xacro">
   <!-- Parámetros generales -->
-  <xacro:property name="package_name" value="my_robot_description"/>
+  <xacro:arg name="package_name" default="my_robot_description"/>
   <!-- Le pasas de donde va a sacar los modelos-->
-  <xacro:property name="mesh_dir" value="meshes"/>
+  <xacro:arg name="mesh_dir" default="meshes"/>
   <!-- Escala global del modelo CAD exportado desde SolidWorks -->
   <xacro:property name="global_scale" value="1.0"/>
@@ -62,5 +62,5 @@
   <xacro:property name="castor_wheel_width" value="0.020"/>
   <xacro:property name="castor_wheel_mass" value="0.086"/>
-  <xacro:include filename="my_robot_gazebo.xacro" />
+  <!-- <xacro:include filename="my_robot_gazebo.xacro" />  Lo saque para probar-->
   <!-- Macros auxiliares -->
   <xacro:macro name="box_inertia" params="m x y z o_xyz o_rpy">
@@ -88,5 +88,5 @@
         <origin xyz="${base_visual_xyz}" rpy="${base_visual_rpy}"/>
         <geometry>
-          <mesh filename="package://${package_name}/${mesh_dir}/${mesh}" scale="${scale}"/>
+          <mesh filename="package://$(arg package_name)/$(arg mesh_dir)/${mesh}" scale="${scale}"/>
         </geometry>
         <material name="blue"/>
@@ -107,5 +107,5 @@
         <origin xyz="${left_wheel_visual_xyz}" rpy="${left_wheel_visual_rpy}"/>
         <geometry>
-          <mesh filename="package://${package_name}/${mesh_dir}/${mesh}" scale="${scale}"/>
+          <mesh filename="package://$(arg package_name)/$(arg mesh_dir)/${mesh}" scale="${scale}"/>
         </geometry>
         <material name="grey"/>
@@ -126,5 +126,5 @@
         <origin xyz="${castor_base_visual_xyz}" rpy="${castor_base_visual_rpy}"/>
         <geometry>
-          <mesh filename="package://${package_name}/${mesh_dir}/${mesh}" scale="${scale}"/>
+          <mesh filename="package://$(arg package_name)/$(arg mesh_dir)/${mesh}" scale="${scale}"/>
         </geometry>
         <material name="green"/>
@@ -138,5 +138,5 @@
         <origin xyz="${castor_wheel_visual_xyz}" rpy="${castor_wheel_visual_rpy}"/>
         <geometry>
-          <mesh filename="package://${package_name}/${mesh_dir}/${mesh}" scale="${scale}"/>
+          <mesh filename="package://$(arg package_name)/$(arg mesh_dir)/${mesh}" scale="${scale}"/>
         </geometry>
         <material name="yellow"/>
@@ -230,4 +230,5 @@
     <child link="Rueda_izquierda_link"/>
     <axis xyz="${left_wheel_axis}"/>
+    <dynamics damping="0.1" friction="0.05"/>
   </joint>
  <!-- Completar Joint rueda_derecha_link>base_link-->
@@ -237,4 +238,5 @@
     <child link="Rueda_derecha_link"/>
     <axis xyz="${right_wheel_axis}"/>
+    <dynamics damping="0.1" friction="0.05"/>
   </joint>
  <!-- Completar Joint Base_castor_link>base_link-->
@@ -251,4 +253,5 @@
     <child link="Rueda_castor_link"/>
     <axis xyz="${castor_wheel_axis}"/>
+    <dynamics damping="0.05" friction="0.02"/>
   </joint>
   <joint name="Lidar_joint" type="fixed">
@@ -258,3 +261,20 @@
     <axis xyz="0 1 0" />
 </joint>
+  <!-- Fricción de las ruedas motrices para reducir deslizamiento en Gazebo -->
+<gazebo reference="Rueda_izquierda_link">
+  <mu1>2.0</mu1>
+  <mu2>2.0</mu2>
+  <kp>1e6</kp>    <kd>1.0</kd>
+</gazebo>
+<gazebo reference="Rueda_derecha_link">
+  <mu1>2.0</mu1>
+  <mu2>2.0</mu2>
+  <kp>1e6</kp>
+  <kd>1.0</kd>
+</gazebo>
+  <!-- Rueda castor con fricción mínima para que gire libre -->
+<gazebo reference="Rueda_castor_link">
+  <mu1>0.01</mu1>
+  <mu2>0.01</mu2>
+</gazebo>
 </robot>

File: src/my_robot_description/urdf/my_robot.urdf.xacro (robot description, xacro)
@@ -3,3 +3,4 @@
     <xacro:include filename="common_properties.xacro" />
     <xacro:include filename="mobile_base.xacro" />
+    <xacro:include filename="my_robot_gazebo.xacro" />
 </robot>

File: src/my_robot_description/urdf/my_robot_gazebo.xacro (robot description, xacro)
@@ -17,13 +17,18 @@
     </gazebo>
     <gazebo>
+        <plugin
+            filename="gz-sim-odometry-publisher-system"
+            name="gz::sim::systems::OdometryPublisher">
+            <odom_frame>odom</odom_frame>
+            <robot_base_frame>base_footprint</robot_base_frame>
+            <dimensions>2</dimensions>
+            <odom_topic>odom_real</odom_topic>
+        </plugin>
+    </gazebo>
+    <gazebo>
         <plugin filename="gz-sim-joint-state-publisher-system" name="gz::sim::systems::JointStatePublisher">
             <joint_name>Rueda_izquierda_joint</joint_name>
             <joint_name>Rueda_derecha_joint</joint_name>
             <joint_name>Rueda_castor_joint</joint_name>
-        </plugin>
-    </gazebo>
-    <gazebo>
-        <plugin filename="gz-sim-sensors-system" name="gz::sim::systems::Sensors">
-            <render_engine>ogre2</render_engine>
         </plugin>
     </gazebo>
